File: AstroPix2/astropix_v2.sch (KiCad schematic (older format))
At the start: 46 parts, among them J1 pcie_GECCO, J10 SPI_right, J3 Vtemp1, J4 SFOut, J5 sample_clock_out, J6 HV_in_external, J8 VBias, J9 SPI_left, U1 TLV333, U2 SN65LVDS4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

Commit message: PCB: First astropix2 layout
Parts:
- removed R13, R14: NC, Resistor_SMD:R_0603_1608Metric, symbol Device:R
- removed R8: 0, Resistor_SMD:R_0603_1608Metric, symbol Device:R
- added C7: .1uF, Capacitor_SMD:C_0603_1608Metric, symbol Device:C
- R15: value 1k -> 2.2k
- R16: value 2k -> 2.2k
- R3, R4: footprint Resistor_SMD:R_0603_1608Metric -> Resistor_SMD:R_0402_1005Metric
- R9: value 680 -> 1k
- renumbered Cvdd3 to C10, Cvdda1 to C11, Cvdda2 to C13, Cvdda3 to C14, Cvdd1 to C8, Cvdd2 to C9
Connections:
- net GND: now also C7.2
- net VDD: now also C7.1
- net HV_in_ext: now reaches J6.1 (In), R1.1, R11.1, R12.1
Changed lines of the file:
@@
 F 0 "R4" H 7920 7146 50  0000 L CNN
 F 1 "100" H 7920 7055 50  0000 L CNN
-F 2 "Resistor_SMD:R_0603_1608Metric" V 7780 7100 50  0001 C CNN
+F 2 "Resistor_SMD:R_0402_1005Metric" V 7780 7100 50  0001 C CNN
 F 3 "~" H 7850 7100 50  0001 C CNN
 	1    7850 7100
@@
 Wire Wire Line
 	8100 7050 8100 6900
-Wire Wire Line
-	8100 6900 7950 6900
 Wire Wire Line
 	8100 7300 8100 7150
@@
 $EndComp
 $Comp
-L Device:C Cvdda1
+L Device:C C11
 U 1 1 6107E1BB
 P 2900 1300
-F 0 "Cvdda1" H 3015 1346 50  0000 L CNN
+F 0 "C11" H 3015 1346 50  0000 L CNN
 F 1 "1nF" H 3015 1255 50  0000 L CNN
 F 2 "Capacitor_SMD:C_0603_1608Metric" H 2938 1150 50  0001 C CNN
@@
 $EndComp
 $Comp
-L Device:C Cvdda2
+L Device:C C13
 U 1 1 6107E1C1
 P 3400 1300
-F 0 "Cvdda2" H 3515 1346 50  0000 L CNN
+F 0 "C13" H 3515 1346 50  0000 L CNN
 F 1 ".1uF" H 3515 1255 50  0000 L CNN
 F 2 "Capacitor_SMD:C_0603_1608Metric" H 3438 1150 50  0001 C CNN
@@
 $EndComp
 $Comp
-L Device:C Cvdda3
+L Device:C C14
 U 1 1 6107E1C7
 P 3900 1300
-F 0 "Cvdda3" H 4015 1346 50  0000 L CNN
+F 0 "C14" H 4015 1346 50  0000 L CNN
 F 1 "10uF" H 4015 1255 50  0000 L CNN
 F 2 "Capacitor_SMD:C_0603_1608Metric" H 3938 1150 50  0001 C CNN
@@
 F 0 "R3" H 6120 9596 50  0000 L CNN
 F 1 "100" H 6120 9505 50  0000 L CNN
-F 2 "Resistor_SMD:R_0603_1608Metric" V 5980 9550 50  0001 C CNN
+F 2 "Resistor_SMD:R_0402_1005Metric" V 5980 9550 50  0001 C CNN
 F 3 "~" H 6050 9550 50  0001 C CNN
 	1    6050 9550
@@
 	6050 9700 6050 9750
 $Comp
-L Device:C Cvdd1
+L Device:C C8
 U 1 1 60D1FE26
 P 1400 1300
-F 0 "Cvdd1" H 1515 1346 50  0000 L CNN
+F 0 "C8" H 1515 1346 50  0000 L CNN
 F 1 "1n" H 1515 1255 50  0000 L CNN
 F 2 "Capacitor_SMD:C_0603_1608Metric" H 1438 1150 50  0001 C CNN
@@
 $EndComp
 $Comp
-L Device:C Cvdd2
+L Device:C C9
 U 1 1 60D1FE2C
 P 1850 1300
-F 0 "Cvdd2" H 1965 1346 50  0000 L CNN
+F 0 "C9" H 1965 1346 50  0000 L CNN
 F 1 ".1uF" H 1965 1255 50  0000 L CNN
 F 2 "Capacitor_SMD:C_0603_1608Metric" H 1888 1150 50  0001 C CNN
@@
 $EndComp
 $Comp
-L Device:C Cvdd3
+L Device:C C10
 U 1 1 60D1FE32
 P 2300 1300
-F 0 "Cvdd3" H 2415 1346 50  0000 L CNN
+F 0 "C10" H 2415 1346 50  0000 L CNN
 F 1 "10uF" H 2415 1255 50  0000 L CNN
 F 2 "Capacitor_SMD:C_0603_1608Metric" H 2338 1150 50  0001 C CNN
@@
 Wire Wire Line
 	12400 6750 12050 6750
-Wire Wire Line
-	7350 9550 7450 9550
 Text Label 9000 8550 0    50   ~ 0
 spi_left_miso1
@@
 	10300 4750 10400 4750
 Connection ~ 10300 4750
-Wire Wire Line
-	12050 7350 12800 7350
 $Comp
 L Device:R R12
@@
 	1    2200 9350
 	1    0    0    -1
-$EndComp
-Wire Wire Line
-	6200 9350 6200 8650
-Wire Wire Line
-	6200 8650 6650 8650
-Connection ~ 6200 9350
-Wire Wire Line
-	6950 8650 7450 8650
-Wire Wire Line
-	7450 8650 7450 9550
-Connection ~ 7450 9550
-$Comp
-L Device:R R8
-U 1 1 611E99CC
-P 6800 8650
-F 0 "R8" V 6593 8650 50  0000 C CNN
-F 1 "0" V 6684 8650 50  0000 C CNN
-F 2 "Resistor_SMD:R_0603_1608Metric" V 6730 8650 50  0001 C CNN
-F 3 "~" H 6800 8650 50  0001 C CNN
-	1    6800 8650
-	0    1    1    0
 $EndComp
 Text Label 800  4950 0    50   ~ 0
@@
 	14550 3450 14100 3450
 Connection ~ 14100 3450
-Wire Wire Line
-	7450 9550 8350 9550
 NoConn ~ 1450 5350
 NoConn ~ 1450 5250
@@
 Wire Wire Line
 	8350 7350 9650 7350
-$Comp
-L Device:R R14
-U 1 1 60E1973A
-P 7950 7500
-F 0 "R14" H 8020 7546 50  0000 L CNN
-F 1 "NC" H 8020 7455 50  0000 L CNN
-F 2 "Resistor_SMD:R_0603_1608Metric" V 7880 7500 50  0001 C CNN
-F 3 "~" H 7950 7500 50  0001 C CNN
-	1    7950 7500
-	1    0    0    -1
-$EndComp
-$Comp
-L Device:R R13
-U 1 1 60E2F145
-P 7950 6700
-F 0 "R13" H 8020 6746 50  0000 L CNN
-F 1 "NC" H 8020 6655 50  0000 L CNN
-F 2 "Resistor_SMD:R_0603_1608Metric" V 7880 6700 50  0001 C CNN
-F 3 "~" H 7950 6700 50  0001 C CNN
-	1    7950 6700
-	1    0    0    -1
-$EndComp
 Wire Wire Line
 	8100 7050 9650 7050
 Wire Wire Line
 	8100 7150 9650 7150
-Wire Wire Line
-	7950 7350 7950 7300
-Connection ~ 7950 7300
-Wire Wire Line
-	7950 7300 8100 7300
-Wire Wire Line
-	7850 7300 7950 7300
-Wire Wire Line
-	7950 6900 7950 6850
-Connection ~ 7950 6900
-Wire Wire Line
-	7950 6900 7850 6900
-$Comp
-L power:VDD #PWR0143
-U 1 1 60ECA3B6
-P 7950 6500
-F 0 "#PWR0143" H 7950 6350 50  0001 C CNN
-F 1 "VDD" H 7965 6673 50  0000 C CNN
-F 2 "" H 7950 6500 50  0001 C CNN
-F 3 "" H 7950 6500 50  0001 C CNN
-	1    7950 6500
-	-1   0    0    -1
-$EndComp
-$Comp
-L power:GNDD #PWR0150
-U 1 1 60EE0C79
-P 7950 7700
-F 0 "#PWR0150" H 7950 7450 50  0001 C CNN
-F 1 "GNDD" H 7954 7545 50  0000 C CNN
-F 2 "" H 7950 7700 50  0001 C CNN
-F 3 "" H 7950 7700 50  0001 C CNN
-	1    7950 7700
-	-1   0    0    -1
-$EndComp
-Wire Wire Line
-	7950 7650 7950 7700
-Wire Wire Line
-	7950 6500 7950 6550
 Text Notes 6600 7550 0    50   ~ 0
 100 Ohm Term\nopt. Failsafe R13=2k R14=4k
@@
 P 14400 4250
 F 0 "R16" V 14193 4250 50  0000 C CNN
-F 1 "2k" V 14284 4250 50  0000 C CNN
+F 1 "2.2k" V 14284 4250 50  0000 C CNN
 F 2 "Resistor_SMD:R_0603_1608Metric" V 14330 4250 50  0001 C CNN
 F 3 "~" H 14400 4250 50  0001 C CNN
@@
 P 13550 3650
 F 0 "R9" V 13343 3650 50  0000 C CNN
-F 1 "680" V 13434 3650 50  0000 C CNN
+F 1 "1k" V 13434 3650 50  0000 C CNN
 F 2 "Resistor_SMD:R_0603_1608Metric" V 13480 3650 50  0001 C CNN
 F 3 "~" H 13550 3650 50  0001 C CNN
@@
 P 13850 4450
 F 0 "R15" H 13920 4496 50  0000 L CNN
-F 1 "1k" H 13920 4405 50  0000 L CNN
+F 1 "2.2k" H 13920 4405 50  0000 L CNN
 F 2 "Resistor_SMD:R_0603_1608Metric" V 13780 4450 50  0001 C CNN
 F 3 "~" H 13850 4450 50  0001 C CNN
@@
 spi_right_miso1
 $Comp
-L power:VDDA #PWR?
+L power:VDDA #PWR0146
 U 1 1 61134A9E
 P 13400 1550
-F 0 "#PWR?" H 13400 1400 50  0001 C CNN
+F 0 "#PWR0146" H 13400 1400 50  0001 C CNN
 F 1 "VDDA" H 13415 1723 50  0000 C CNN
 F 2 "" H 13400 1550 50  0001 C CNN
@@
 $EndComp
 $Comp
-L power:VDDA #PWR?
+L power:VDDA #PWR0148
 U 1 1 6114F02E
 P 13050 4000
-F 0 "#PWR?" H 13050 3850 50  0001 C CNN
+F 0 "#PWR0148" H 13050 3850 50  0001 C CNN
 F 1 "VDDA" H 13065 4173 50  0000 C CNN
 F 2 "" H 13050 4000 50  0001 C CNN
@@
 	1    0    0    -1
 $EndComp
+$Comp
+L power:VDD #PWR0152
+U 1 1 60E7BEA5
+P 5200 8200
+F 0 "#PWR0152" H 5200 8050 50  0001 C CNN
+F 1 "VDD" H 5215 8373 50  0000 C CNN
+F 2 "" H 5200 8200 50  0001 C CNN
+F 3 "" H 5200 8200 50  0001 C CNN
+	1    5200 8200
+	-1   0    0    -1
+$EndComp
+$Comp
+L Device:C C7
+U 1 1 60E7BEAB
+P 5200 8450
+F 0 "C7" H 5315 8496 50  0000 L CNN
+F 1 ".1uF" H 5315 8405 50  0000 L CNN
+F 2 "Capacitor_SMD:C_0603_1608Metric" H 5238 8300 50  0001 C CNN
+F 3 "~" H 5200 8450 50  0001 C CNN
+	1    5200 8450
+	1    0    0    -1
+$EndComp
+$Comp
+L power:GNDD #PWR0153
+U 1 1 60E7BEB1
+P 5200 8700
+F 0 "#PWR0153" H 5200 8450 50  0001 C CNN
+F 1 "GNDD" H 5204 8545 50  0000 C CNN
+F 2 "" H 5200 8700 50  0001 C CNN
+F 3 "" H 5200 8700 50  0001 C CNN
+	1    5200 8700
+	-1   0    0    -1
+$EndComp
+Wire Wire Line
+	5200 8600 5200 8700
+Wire Wire Line
+	5200 8200 5200 8300
+Wire Wire Line
+	7850 6900 8100 6900
+Wire Wire Line
+	7850 7300 8100 7300
+Wire Wire Line
+	7350 9550 8350 9550
+Wire Wire Line
+	10800 4600 10800 4750
+Wire Wire Line
+	10800 4750 10700 4750
+Connection ~ 10700 4750
+Wire Wire Line
+	12050 7350 12800 7350
+Text Label 5250 1700 0    50   ~ 0
+HV_in_ext
 $EndSCHEMATC

Commit message: PCB: Updated astropix2 pcb
-diff pair impedance
-added teardropds
-small fixes
Parts:
- added Logo2: HV_logo, astropix:hv, symbol astropix:HV_logo
- C3, C4, C5, C6: Voltage (none) -> 250V
- C8: value 1n -> 1nF
Changed lines of the file:
@@
 F 2 "Capacitor_SMD:C_1210_3225Metric" H 6538 750 50  0001 C CNN
 F 3 "~" H 6500 900 50  0001 C CNN
+F 4 "250V" H 6500 900 50  0001 C CNN "Voltage"
 	1    6500 900
 	1    0    0    -1
@@
 F 2 "Capacitor_SMD:C_1210_3225Metric" H 6938 750 50  0001 C CNN
 F 3 "~" H 6900 900 50  0001 C CNN
+F 4 "250V" H 6900 900 50  0001 C CNN "Voltage"
 	1    6900 900
 	1    0    0    -1
@@
 F 2 "Capacitor_SMD:C_1210_3225Metric" H 6538 1650 50  0001 C CNN
 F 3 "~" H 6500 1800 50  0001 C CNN
+F 4 "250V" H 6500 1800 50  0001 C CNN "Voltage"
 	1    6500 1800
 	1    0    0    -1
@@
 F 2 "Capacitor_SMD:C_1210_3225Metric" H 6938 1650 50  0001 C CNN
 F 3 "~" H 6900 1800 50  0001 C CNN
+F 4 "250V" H 6900 1800 50  0001 C CNN "Voltage"
 	1    6900 1800
 	1    0    0    -1
@@
 P 1400 1300
 F 0 "C8" H 1515 1346 50  0000 L CNN
-F 1 "1n" H 1515 1255 50  0000 L CNN
+F 1 "1nF" H 1515 1255 50  0000 L CNN
 F 2 "Capacitor_SMD:C_0603_1608Metric" H 1438 1150 50  0001 C CNN
 F 3 "~" H 1400 1300 50  0001 C CNN
@@
 Text Label 9000 8550 0    50   ~ 0
 spi_left_miso1
-Text Label 9000 8850 0    50   ~ 0
-spi_left_clk
-Text Label 9000 8950 0    50   ~ 0
-spi_left_csn
 Text Label 9000 8650 0    50   ~ 0
 spi_left_miso0
@@
 Wire Wire Line
 	9000 8750 9650 8750
-Wire Wire Line
-	9000 8850 9650 8850
-Wire Wire Line
-	9000 8950 9650 8950
 Text Label 12700 8550 2    50   ~ 0
 spi_right_miso1
@@
 Text Label 800  4950 0    50   ~ 0
 spi_left_miso1
-Text Label 800  4750 0    50   ~ 0
-spi_left_clk
-Text Label 800  4850 0    50   ~ 0
-spi_left_csn
 Text Label 800  5050 0    50   ~ 0
 spi_left_miso0
@@
 Wire Wire Line
 	800  5150 1450 5150
-Wire Wire Line
-	800  4750 1450 4750
-Wire Wire Line
-	800  4850 1450 4850
 Wire Wire Line
 	14100 1950 14100 2000
@@
 Text Label 12150 2300 0    50   ~ 0
 VPBias
-$Comp
-L astropix:KIT_logo Logo1
-U 1 1 6167E799
-P 2550 10100
-F 0 "Logo1" H 2350 10250 50  0000 L CNN
-F 1 "KIT_logo" H 2400 10100 50  0000 L CNN
-F 2 "astropix:logo" H 2550 10100 50  0001 C CNN
-F 3 "" H 2550 10100 50  0001 C CNN
-	1    2550 10100
-	1    0    0    -1
-$EndComp
 NoConn ~ 12050 7850
 NoConn ~ 1450 5450
@@
 Wire Wire Line
 	12050 7350 12800 7350
+Wire Wire Line
+	9000 8950 9650 8950
+Text Label 9000 8950 0    50   ~ 0
+spi_left_csn
+Wire Wire Line
+	9000 8850 9650 8850
+Text Label 9000 8850 0    50   ~ 0
+spi_left_clk
 Text Label 5250 1700 0    50   ~ 0
 HV_in_ext
+Text Label 800  4750 0    50   ~ 0
+spi_left_csn
+Wire Wire Line
+	800  4750 1450 4750
+Text Label 800  4850 0    50   ~ 0
+spi_left_clk
+Wire Wire Line
+	800  4850 1450 4850
+$Comp
+L astropix:KIT_logo Logo1
+U 1 1 6167E799
+P 2550 10100
+F 0 "Logo1" H 2350 10250 50  0000 L CNN
+F 1 "KIT_logo" H 2400 10100 50  0000 L CNN
+F 2 "astropix:logo" H 2550 10100 50  0001 C CNN
+F 3 "" H 2550 10100 50  0001 C CNN
+	1    2550 10100
+	1    0    0    -1
+$EndComp
+$Comp
+L astropix:HV_logo Logo2
+U 1 1 610D1472
+P 2550 10450
+F 0 "Logo2" H 2350 10600 50  0000 L CNN
+F 1 "HV_logo" H 2400 10450 50  0000 L CNN
+F 2 "astropix:hv" H 2550 10450 50  0001 C CNN
+F 3 "" H 2550 10450 50  0001 C CNN
+	1    2550 10450
+	1    0    0    -1
+$EndComp
 $EndSCHEMATC

Commit message: PCB: Small corrections
Parts:
- removed J8: VBias, Connector_PinHeader_2.54mm:PinHeader_1x03_P2.54mm_Vertical, symbol Connector_Generic:Conn_01x03
Connections:
- net labels removed: VPBias, pamp
- wire segments 295 -> 291
- no-connect marks 61 -> 63
Other:
- note removed: "Remove?"
Changed lines of the file:
@@
 Text Label 12350 3650 2    50   ~ 0
 Vtemp1
-$Comp
-L Connector_Generic:Conn_01x03 J8
-U 1 1 60D156C8
-P 12600 2300
-F 0 "J8" H 12518 2617 50  0000 C CNN
-F 1 "VBias" H 12518 2526 50  0000 C CNN
-F 2 "Connector_PinHeader_2.54mm:PinHeader_1x03_P2.54mm_Vertical" H 12600 2300 50  0001 C CNN
-F 3 "~" H 12600 2300 50  0001 C CNN
-	1    12600 2300
-	1    0    0    -1
-$EndComp
-Wire Wire Line
-	12400 2200 12050 2200
-Wire Wire Line
-	12050 2300 12400 2300
-$Comp
-L power:GNDA #PWR0142
-U 1 1 60D3AC50
-P 12300 2450
-F 0 "#PWR0142" H 12300 2200 50  0001 C CNN
-F 1 "GNDA" H 12305 2277 50  0000 C CNN
-F 2 "" H 12300 2450 50  0001 C CNN
-F 3 "" H 12300 2450 50  0001 C CNN
-	1    12300 2450
-	-1   0    0    -1
-$EndComp
-Wire Wire Line
-	12400 2400 12300 2400
-Wire Wire Line
-	12300 2400 12300 2450
 Text Label 14450 7650 0    50   ~ 0
 spi_left_miso1
@@
 	3400 1550 3900 1550
 Connection ~ 3400 1550
-Text Label 12150 2200 0    50   ~ 0
-pamp
-Text Label 12150 2300 0    50   ~ 0
-VPBias
 NoConn ~ 12050 7850
 NoConn ~ 1450 5450
-Text Notes 12500 2550 0    50   ~ 0
-Remove?
 $Comp
 L Device:R R16
@@
 	1    0    0    -1
 $EndComp
+NoConn ~ 12050 2200
+NoConn ~ 12050 2300
 $EndSCHEMATC

Commit message: PCB: Apix v2 updates
- Added SPI series resistors
- connected spi_right_clk to FMC
- Updated Amplifier Layout
Parts:
- added R10, R13, R14, R17, R18, R8: 22, Resistor_SMD:R_0402_1005Metric, symbol Device:R
- R6: value 22 -> 47
Connections:
- wire segments 291 -> 298
- no-connect marks 63 -> 62
Other:
- moved on the sheet: J5
Changed lines of the file:
@@
 Wire Wire Line
 	12400 6750 12050 6750
-Text Label 9000 8550 0    50   ~ 0
+Text Label 8300 8550 0    50   ~ 0
 spi_left_miso1
-Text Label 9000 8650 0    50   ~ 0
+Text Label 8300 8650 0    50   ~ 0
 spi_left_miso0
-Text Label 9000 8750 0    50   ~ 0
+Text Label 9150 8750 0    50   ~ 0
 spi_left_mosi
-Wire Wire Line
-	9000 8550 9650 8550
-Wire Wire Line
-	9000 8650 9650 8650
-Wire Wire Line
-	9000 8750 9650 8750
 Text Label 12700 8550 2    50   ~ 0
 spi_right_miso1
-Text Label 12700 8850 2    50   ~ 0
+Text Label 13600 8850 2    50   ~ 0
 spi_right_clk
 Text Label 12700 8950 2    50   ~ 0
@@
 Text Label 12700 8650 2    50   ~ 0
 spi_right_miso0
-Text Label 12700 8750 2    50   ~ 0
+Text Label 13600 8750 2    50   ~ 0
 spi_right_mosi
-Wire Wire Line
-	12700 8550 12050 8550
-Wire Wire Line
-	12700 8650 12050 8650
-Wire Wire Line
-	12700 8750 12050 8750
-Wire Wire Line
-	12700 8850 12050 8850
-Wire Wire Line
-	12700 8950 12050 8950
-Text Label 12650 7350 2    50   ~ 0
+Text Label 12850 7350 2    50   ~ 0
 sc_out
 Text Label 8200 9550 2    50   ~ 0
@@
 L Connector:Conn_Coaxial J5
 U 1 1 60F540B4
-P 13000 7350
-F 0 "J5" H 13100 7325 50  0000 L CNN
-F 1 "sample_clock_out" H 13100 7234 50  0000 L CNN
-F 2 "Connector_Coaxial:SMA_Molex_73251-2200_Horizontal" H 13000 7350 50  0001 C CNN
-F 3 " ~" H 13000 7350 50  0001 C CNN
-	1    13000 7350
-	1    0    0    -1
-$EndComp
-Wire Wire Line
-	13000 7550 13000 7650
+P 13200 7350
+F 0 "J5" H 13300 7325 50  0000 L CNN
+F 1 "sample_clock_out" H 13300 7234 50  0000 L CNN
+F 2 "Connector_Coaxial:SMA_Molex_73251-2200_Horizontal" H 13200 7350 50  0001 C CNN
+F 3 " ~" H 13200 7350 50  0001 C CNN
+	1    13200 7350
+	1    0    0    -1
+$EndComp
+Wire Wire Line
+	13200 7550 13200 7650
 $Comp
 L Mechanical:MountingHole H1
@@
 NoConn ~ 1450 7750
 NoConn ~ 1450 7650
-NoConn ~ 1450 7550
 NoConn ~ 1450 6050
 NoConn ~ 1450 6150
@@
 L power:GNDD #PWR0136
 U 1 1 6168FAAD
-P 13000 7650
-F 0 "#PWR0136" H 13000 7400 50  0001 C CNN
-F 1 "GNDD" H 13004 7495 50  0000 C CNN
-F 2 "" H 13000 7650 50  0001 C CNN
-F 3 "" H 13000 7650 50  0001 C CNN
-	1    13000 7650
+P 13200 7650
+F 0 "#PWR0136" H 13200 7400 50  0001 C CNN
+F 1 "GNDD" H 13204 7495 50  0000 C CNN
+F 2 "" H 13200 7650 50  0001 C CNN
+F 3 "" H 13200 7650 50  0001 C CNN
+	1    13200 7650
 	-1   0    0    -1
 $EndComp
@@
 P 14850 2300
 F 0 "R6" V 14643 2300 50  0000 C CNN
-F 1 "22" V 14734 2300 50  0000 C CNN
+F 1 "47" V 14734 2300 50  0000 C CNN
 F 2 "Resistor_SMD:R_0603_1608Metric" V 14780 2300 50  0001 C CNN
 F 3 "~" H 14850 2300 50  0001 C CNN
@@
 	10300 900  10300 1100
 Wire Wire Line
-	8350 9550 8350 7350
-Wire Wire Line
-	8350 7350 9650 7350
+	8200 9550 8200 7350
+Wire Wire Line
+	8200 7350 9650 7350
 Wire Wire Line
 	8100 7050 9650 7050
@@
 L power:GNDD #PWR0140
 U 1 1 611F5306
-P 9350 8250
-F 0 "#PWR0140" H 9350 8000 50  0001 C CNN
-F 1 "GNDD" H 9354 8095 50  0000 C CNN
-F 2 "" H 9350 8250 50  0001 C CNN
-F 3 "" H 9350 8250 50  0001 C CNN
-	1    9350 8250
+P 9250 8250
+F 0 "#PWR0140" H 9250 8000 50  0001 C CNN
+F 1 "GNDD" H 9254 8095 50  0000 C CNN
+F 2 "" H 9250 8250 50  0001 C CNN
+F 3 "" H 9250 8250 50  0001 C CNN
+	1    9250 8250
 	-1   0    0    -1
 $EndComp
 Wire Wire Line
-	9350 8250 9350 8200
-Wire Wire Line
-	9350 8200 9650 8200
+	9250 8250 9250 8200
+Wire Wire Line
+	9250 8200 9650 8200
 $Comp
 L astropix:pcie_GECCO J1
@@
 NoConn ~ 3200 7150
 Wire Wire Line
+	800  7550 1450 7550
+Wire Wire Line
 	800  7450 1450 7450
 Wire Wire Line
@@
 Wire Wire Line
 	800  7250 1450 7250
-Wire Wire Line
-	800  7150 1450 7150
+Text Label 800  7550 0    50   ~ 0
+spi_right_mosi
+Text Label 800  7350 0    50   ~ 0
+spi_right_miso0
 Text Label 800  7450 0    50   ~ 0
-spi_right_mosi
+spi_right_csn
 Text Label 800  7250 0    50   ~ 0
-spi_right_miso0
-Text Label 800  7350 0    50   ~ 0
-spi_right_csn
-Text Label 800  7150 0    50   ~ 0
 spi_right_miso1
 $Comp
@@
 	7850 7300 8100 7300
 Wire Wire Line
-	7350 9550 8350 9550
+	7350 9550 8200 9550
 Wire Wire Line
 	10800 4600 10800 4750
@@
 	10800 4750 10700 4750
 Connection ~ 10700 4750
-Wire Wire Line
-	12050 7350 12800 7350
-Wire Wire Line
-	9000 8950 9650 8950
-Text Label 9000 8950 0    50   ~ 0
+Text Label 8300 8950 0    50   ~ 0
 spi_left_csn
-Wire Wire Line
-	9000 8850 9650 8850
-Text Label 9000 8850 0    50   ~ 0
+Text Label 9150 8850 0    50   ~ 0
 spi_left_clk
 Text Label 5250 1700 0    50   ~ 0
@@
 NoConn ~ 12050 2200
 NoConn ~ 12050 2300
+$Comp
+L Device:R R8
+U 1 1 60F78001
+P 12250 7350
+F 0 "R8" V 12043 7350 50  0000 C CNN
+F 1 "22" V 12134 7350 50  0000 C CNN
+F 2 "Resistor_SMD:R_0402_1005Metric" V 12180 7350 50  0001 C CNN
+F 3 "~" H 12250 7350 50  0001 C CNN
+	1    12250 7350
+	0    1    1    0
+$EndComp
+Wire Wire Line
+	12400 7350 13000 7350
+Wire Wire Line
+	12050 7350 12100 7350
+$Comp
+L Device:R R10
+U 1 1 60FC84E9
+P 9000 8550
+F 0 "R10" V 8900 8550 50  0000 C CNN
+F 1 "22" V 9000 8550 50  0000 C CNN
+F 2 "Resistor_SMD:R_0402_1005Metric" V 8930 8550 50  0001 C CNN
+F 3 "~" H 9000 8550 50  0001 C CNN
+	1    9000 8550
+	0    1    1    0
+$EndComp
+Wire Wire Line
+	9150 8550 9650 8550
+Wire Wire Line
+	8300 8550 8850 8550
+$Comp
+L Device:R R13
+U 1 1 6102DFC2
+P 9000 8650
+F 0 "R13" V 9100 8650 50  0000 C CNN
+F 1 "22" V 9000 8650 50  0000 C CNN
+F 2 "Resistor_SMD:R_0402_1005Metric" V 8930 8650 50  0001 C CNN
+F 3 "~" H 9000 8650 50  0001 C CNN
+	1    9000 8650
+	0    1    1    0
+$EndComp
+Wire Wire Line
+	8300 8650 8850 8650
+Wire Wire Line
+	9150 8650 9650 8650
+Wire Wire Line
+	9150 8750 9650 8750
+Wire Wire Line
+	9150 8850 9650 8850
+$Comp
+L Device:R R14
+U 1 1 610ACEEF
+P 9000 8950
+F 0 "R14" V 9100 8950 50  0000 C CNN
+F 1 "22" V 9000 8950 50  0000 C CNN
+F 2 "Resistor_SMD:R_0402_1005Metric" V 8930 8950 50  0001 C CNN
+F 3 "~" H 9000 8950 50  0001 C CNN
+	1    9000 8950
+	0    1    1    0
+$EndComp
+Wire Wire Line
+	8300 8950 8850 8950
+Wire Wire Line
+	9150 8950 9650 8950
+$Comp
+L Device:R R17
+U 1 1 610FAFC8
+P 12900 8750
+F 0 "R17" V 12800 8750 50  0000 C CNN
+F 1 "22" V 12900 8750 50  0000 C CNN
+F 2 "Resistor_SMD:R_0402_1005Metric" V 12830 8750 50  0001 C CNN
+F 3 "~" H 12900 8750 50  0001 C CNN
+	1    12900 8750
+	0    1    1    0
+$EndComp
+$Comp
+L Device:R R18
+U 1 1 610FB87E
+P 12900 8850
+F 0 "R18" V 13000 8850 50  0000 C CNN
+F 1 "22" V 12900 8850 50  0000 C CNN
+F 2 "Resistor_SMD:R_0402_1005Metric" V 12830 8850 50  0001 C CNN
+F 3 "~" H 12900 8850 50  0001 C CNN
+	1    12900 8850
+	0    1    1    0
+$EndComp
+Wire Wire Line
+	12050 8850 12750 8850
+Wire Wire Line
+	13050 8850 13600 8850
+Wire Wire Line
+	12050 8950 12700 8950
+Wire Wire Line
+	12050 8750 12750 8750
+Wire Wire Line
+	13050 8750 13600 8750
+Wire Wire Line
+	12050 8650 12700 8650
+Wire Wire Line
+	12050 8550 12700 8550
+Wire Wire Line
+	800  7150 1450 7150
+Text Label 800  7150 0    50   ~ 0
+spi_right_clk
 $EndSCHEMATC

Commit message: PCB: Added holes for HIT bonding fixture
Parts:
- added H3: bonder, astropix:bonder, symbol astropix:bonder
Changed lines of the file:
@@
 Text Label 800  7150 0    50   ~ 0
 spi_right_clk
+$Comp
+L astropix:bonder H3
+U 1 1 6106C8E5
+P 1500 10400
+F 0 "H3" H 1350 10550 50  0000 L CNN
+F 1 "bonder" H 1350 10400 50  0000 L CNN
+F 2 "astropix:bonder" H 1500 10400 50  0001 C CNN
+F 3 "" H 1500 10400 50  0001 C CNN
+	1    1500 10400
+	1    0    0    -1
+$EndComp
 $EndSCHEMATC
