File: AstroPix2/astropix_v2.sch (KiCad schematic (older format))
At the start: 51 parts, among them J1 pcie_GECCO, J10 SPI_right, J3 Vtemp1, J4 SFOut, J5 sample_clock_out, J6 HV_in_external, J9 SPI_left, U1 TLV333, U2 SN65LVDS4, U3 OPA320S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

Commit message: PCB V2: Connected SR_out/RB + Updated production files
Connections:
- net labels added: sr_out, sr_rb
- wire segments 298 -> 300
- no-connect marks 62 -> 59
Changed lines of the file:
@@
 NoConn ~ 1450 3450
 Wire Wire Line
-	9650 7800 9350 7800
-Wire Wire Line
 	9650 7900 9350 7900
 Wire Wire Line
@@
 Wire Wire Line
 	9650 8100 9350 8100
-Text Label 9350 7800 0    50   ~ 0
-sr_ck1
 Text Label 9350 7900 0    50   ~ 0
 sr_ck2
@@
 	1400 1050 1400 1150
 Wire Wire Line
+	3200 5450 3900 5450
+Text Label 3900 5450 2    50   ~ 0
+res_n
+Wire Wire Line
 	3200 5350 3900 5350
 Text Label 3900 5350 2    50   ~ 0
-res_n
-Wire Wire Line
-	3200 5250 3900 5250
-Text Label 3900 5250 2    50   ~ 0
 interrupt
 Text Label 3800 6350 2    50   ~ 0
@@
 Wire Wire Line
 	3200 4950 3900 4950
+Text Label 3900 5250 2    50   ~ 0
+timestamp_clk
+Wire Wire Line
+	3900 5250 3200 5250
 Text Label 3900 5150 2    50   ~ 0
-timestamp_clk
+hold
 Wire Wire Line
 	3900 5150 3200 5150
-Text Label 3900 5450 2    50   ~ 0
-hold
-Wire Wire Line
-	3900 5450 3200 5450
-NoConn ~ 1450 5750
 NoConn ~ 1450 5850
 NoConn ~ 3200 5750
@@
 	14550 3450 14100 3450
 Connection ~ 14100 3450
-NoConn ~ 1450 5350
-NoConn ~ 1450 5250
 Wire Wire Line
 	13600 3300 13600 2200
@@
 	3400 1550 3900 1550
 Connection ~ 3400 1550
-NoConn ~ 12050 7850
-NoConn ~ 1450 5450
 $Comp
 L Device:R R16
@@
 Text Notes 5000 850  0    50   ~ 0
 GECCO HV Clearance?\n
-$Comp
-L power:GNDD #PWR0140
-U 1 1 611F5306
-P 9250 8250
-F 0 "#PWR0140" H 9250 8000 50  0001 C CNN
-F 1 "GNDD" H 9254 8095 50  0000 C CNN
-F 2 "" H 9250 8250 50  0001 C CNN
-F 3 "" H 9250 8250 50  0001 C CNN
-	1    9250 8250
-	-1   0    0    -1
-$EndComp
-Wire Wire Line
-	9250 8250 9250 8200
-Wire Wire Line
-	9250 8200 9650 8200
 $Comp
 L astropix:pcie_GECCO J1
@@
 	1    0    0    -1
 $EndComp
+NoConn ~ 1450 5250
+NoConn ~ 1450 5750
+Text Label 9350 7800 0    50   ~ 0
+sr_ck1
+Wire Wire Line
+	9650 7800 9350 7800
+Text Label 12350 7850 2    50   ~ 0
+sr_out
+Wire Wire Line
+	12350 7850 12050 7850
+Wire Wire Line
+	9650 8200 9350 8200
+Text Label 9350 8200 0    50   ~ 0
+sr_rb
+Text Label 1150 5350 0    50   ~ 0
+sr_out
+Wire Wire Line
+	1450 5350 1150 5350
+Wire Wire Line
+	1450 5450 1150 5450
+Text Label 1150 5450 0    50   ~ 0
+sr_rb
 $EndSCHEMATC
