File: AstroPix4/astropix_v4.kicad_pcb (KiCad board)
At the start: 4 copper layers, 51.3 x 48.9 mm, 36 parts, among them J1 pcie_GECCO, J10 SPI_right, J11 HV, J2 Conn_02x04_Odd_Even, J4 SFOut, J6 HV_in_external, J8 HBOut, J9 SPI_left, U1 AstroPix4_split_powerring

Commit message: PCB: AstroPix4 v1 \w production files + bondplan
Parts:
- added Logo3: HV_logo, astropix:hv, F.Cu at (1.77, 1.47)
