File: AstroPix4/astropix_v4.kicad_sch (KiCad schematic)
At the start: 37 parts, among them J1 pcie_GECCO, J10 SPI_right, J11 HV, J2 Conn_02x04_Odd_Even, J4 SFOut, J6 HV_in_external, J8 HBOut, J9 SPI_left, U1 AstroPix4_split_powerring

Commit message: PCB: AstroPix4 v1 \w production files + bondplan
Connections:
- net GND: no longer U1.B36 (gnda!)
- no-connect marks 57 -> 55
Changed lines of the file:
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@@
   (junction (at 363.22 335.28) (diameter 0) (color 0 0 0 0)
-  )
-  (junction (at 360.68 200.66) (diameter 0) (color 0 0 0 0)
   )
   (junction (at 513.08 121.92) (diameter 0) (color 0 0 0 0)
@@
   (no_connect (at 93.98 168.91))
   (no_connect (at 93.98 232.41))
-  (no_connect (at 322.58 147.32))
   (no_connect (at 138.43 242.57))
   (no_connect (at 93.98 143.51))
@@
   (no_connect (at 138.43 234.95))
   (no_connect (at 93.98 255.27))
-  (no_connect (at 408.94 101.6))
   (no_connect (at 138.43 171.45))
   (no_connect (at 93.98 257.81))
@@
     (stroke (width 0) (type default))
   )
-  (wire (pts (xy 360.68 200.66) (xy 363.22 200.66))
+  (wire (pts (xy 358.14 200.66) (xy 363.22 200.66))
     (stroke (width 0) (type default))
   )
@@
     (stroke (width 0) (type default))
   )
-  (wire (pts (xy 360.68 196.85) (xy 360.68 200.66))
-    (stroke (width 0) (type default))
-  )
   (wire (pts (xy 467.36 297.18) (xy 483.87 297.18))
     (stroke (width 0) (type default))
@@
   )
   (wire (pts (xy 77.47 250.19) (xy 93.98 250.19))
-    (stroke (width 0) (type default))
-  )
-  (wire (pts (xy 358.14 200.66) (xy 360.68 200.66))
     (stroke (width 0) (type default))
   )
@@
     (pin "B12")
     (pin "B13")
-    (pin "B2")
     (pin "B3")
-    (pin "B36")
     (pin "B37")
     (pin "B38")
@@
     (pin "B63")
     (pin "B66")
-    (pin "B67")
     (pin "B68")
     (pin "B71")
@@
     (pin "B12")
     (pin "B13")
-    (pin "B2")
     (pin "B3")
-    (pin "B36")
     (pin "B37")
     (pin "B38")
@@
     (pin "B63")
     (pin "B66")
-    (pin "B67")
     (pin "B68")
     (pin "B71")
